File: 24512/24512.sch (KiCad schematic (older format))
At the start: 15 parts, among them J1 Conn_01x05, U1 24LC1025

Commit message: Part Numbers added
Parts:
- U1: Part (none) -> C79986
Changed lines of the file:
@@
 F 2 "Package_SO:SOIC-8_3.9x4.9mm_P1.27mm" H 4300 2200 50  0001 C CNN
 F 3 "http://ww1.microchip.com/downloads/en/DeviceDoc/21941B.pdf" H 4300 2200 50  0001 C CNN
+F 4 "C79986" H 4300 2200 50  0001 C CNN "Part"
 	1    4300 2200
 	1    0    0    -1
