File: MB85RS256V/MB85RS256V.sch (KiCad schematic (older format))
At the start: 6 parts, among them J1 Conn_01x08, U1 MB85RS64

Commit message: Part Numbers added
Parts:
- U1: Part (none) -> C8742
Changed lines of the file:
@@
 F 2 "Package_SO:SOIC-8_3.9x4.9mm_P1.27mm" H 3800 2000 50  0001 C CNN
 F 3 "http://www.fujitsu.com/downloads/MICRO/fme/fram/datasheet-MB85RS64.pdf" H 3800 2000 50  0001 C CNN
+F 4 "C8742" H 4150 2050 50  0001 C CNN "Part"
 	1    4150 2050
 	1    0    0    -1
