File: 24LCXXX/24LCXXX.sch (KiCad schematic (older format))
At the start: 15 parts, among them J1 Conn_01x05, U1 24LC1025

Commit message: 24LCXXX Added in place of 24512
Parts:
- U1: value 24LC1025 -> 24LCXXX; Part (none) -> C79986
Changed lines of the file:
@@
 encoding utf-8
 Sheet 1 1
-Title "24LC512 Based EEPROM Module"
+Title "24LCXXX Based EEPROM Module"
 Date "2019-12-05"
 Rev "1"
@@
 Comment1 "SirBoard"
 Comment2 "SirKeep"
-Comment3 "24LC512"
+Comment3 "24LC64, 24LC128, 24LC256, 24LC512, 24LC1024"
 Comment4 ""
 $EndDescr
@@
 P 4300 2200
 F 0 "U1" H 4300 2678 50  0000 C CNN
-F 1 "24LC1025" H 4300 2588 50  0000 C CNN
+F 1 "24LCXXX" H 4300 2588 50  0000 C CNN
 F 2 "Package_SO:SOIC-8_3.9x4.9mm_P1.27mm" H 4300 2200 50  0001 C CNN
 F 3 "http://ww1.microchip.com/downloads/en/DeviceDoc/21941B.pdf" H 4300 2200 50  0001 C CNN
+F 4 "C79986" H 4300 2200 50  0001 C CNN "Part"
 	1    4300 2200
 	1    0    0    -1

Commit message: Part numbers added for all variants
Parts:
- U1: Part C79986 -> C7999; C79984; C79989; C79990; C79991
Changed lines of the file:
@@
 EESchema Schematic File Version 4
-LIBS:24512-cache
+LIBS:24LCXXX-cache
 EELAYER 29 0
 EELAYER END
@@
 F 2 "Package_SO:SOIC-8_3.9x4.9mm_P1.27mm" H 4300 2200 50  0001 C CNN
 F 3 "http://ww1.microchip.com/downloads/en/DeviceDoc/21941B.pdf" H 4300 2200 50  0001 C CNN
-F 4 "C79986" H 4300 2200 50  0001 C CNN "Part"
+F 4 "C7999; C79984; C79989; C79990; C79991" H 4300 2200 50  0001 C CNN "Part"
 	1    4300 2200
 	1    0    0    -1
