File: MB85RSXXX/MB85RSXXX.sch (KiCad schematic (older format))
At the start: 6 parts, among them J1 Conn_01x08, U1 MB85RS64

Commit message: MB85RSXXX Added in place of MB85RS256
Parts:
- U1: Part (none) -> C8742
Changed lines of the file:
@@
 encoding utf-8
 Sheet 1 1
-Title "MB85RS256B Based FRAM Module"
+Title "MB85RSXXX Based FRAM Module"
 Date "2019-12-06"
 Rev "1"
@@
 Comment1 "SirBoard"
 Comment2 "SirKeep"
-Comment3 "MB85RS256B"
+Comment3 "MB85RS16, MB85RS64, MB85RS128, MB85RS256, MB85RS512, MB85RS1M"
 Comment4 ""
 $EndDescr
@@
 F 2 "Package_SO:SOIC-8_3.9x4.9mm_P1.27mm" H 3800 2000 50  0001 C CNN
 F 3 "http://www.fujitsu.com/downloads/MICRO/fme/fram/datasheet-MB85RS64.pdf" H 3800 2000 50  0001 C CNN
+F 4 "C8742" H 4150 2050 50  0001 C CNN "Part"
 	1    4150 2050
 	1    0    0    -1

Commit message: Part numbers added for all variants
Parts:
- U1: Part C8742 -> C38647; C8741; C126732; C8742; C93052; C126733
Changed lines of the file:
@@
 EESchema Schematic File Version 4
-LIBS:MB85RS256V-cache
+LIBS:MB85RSXXX-cache
 EELAYER 29 0
 EELAYER END
@@
 F 2 "Package_SO:SOIC-8_3.9x4.9mm_P1.27mm" H 3800 2000 50  0001 C CNN
 F 3 "http://www.fujitsu.com/downloads/MICRO/fme/fram/datasheet-MB85RS64.pdf" H 3800 2000 50  0001 C CNN
-F 4 "C8742" H 4150 2050 50  0001 C CNN "Part"
+F 4 "C38647; C8741; C126732; C8742; C93052; C126733" H 4150 2050 50  0001 C CNN "Part"
 	1    4150 2050
 	1    0    0    -1
